Commit message: updated bringup and configs

File: src/nova_nav/urdf/nova_agv.urdf (robot description, URDF)
Before this commit: robot nova_nav, 13 links, 12 joints
Links:
- removed link scan_link
- added link laser_frame, mass 1e-5; collision box size=.1 .1 .1; visual mesh filename=package://nova_nav/meshes/lidar.stl
Joints:
- removed joint KITI UTAMA
- removed joint scan_joint
- added joint KIRI_UTAMA: type continuous, parent base_link, child KIRI_UTAMA, origin xyz=-0.0015818 -0.1135 -0.19675 rpy=3.1416 0 0, axis 0 0 1, limit effort=50 velocity=50
- added joint laser_joint: type fixed, parent base_link, child laser_frame, origin xyz=0.245 0.05 0 rpy=0 0 0, axis 0 1 0

Commit message: m-explore and correct orentation

File: src/nova_nav/urdf/nova_agv.urdf (robot description, URDF)
Before this commit: robot nova_nav, 13 links, 12 joints
Joints:
- joint laser_joint: axis 0 1 0 -> 0 0 0; origin xyz=0.245 0.05 0 rpy=0 0 0 -> xyz=-0.245 0.05 0 rpy=-1.5708 0 0
