Commit message: kinematic test1

File: src/nova_arm/urdf/nova_arm.urdf (robot description, URDF)
Before this commit: robot nova_arm, 6 links, 5 joints
Joints:
- joint joint_1: axis 0 1 0 -> 0 0 1; origin xyz=0 0  0.065125 rpy=1.5708 0 0.0056739 -> xyz=0 0  0.085 rpy=0 0 0
- joint joint_2: axis 0 1 0 -> 0 0 1; origin xyz=0 0.066 0 rpy=1.5708 0 0 -> xyz=0 0 0.066 rpy=0 -1.5708 0
- joint joint_3: axis 0 1 0 -> 0 0 1; limit lower=-4.0 upper=0.9 effort=10 velocity=1.5 -> lower=-2.332 upper=2.332 effort=10 velocity=1.5; origin xyz=0 0 -0.2 rpy=3.1416 0 3.1416 -> xyz=0.20 0 0 rpy=0 0 0
- joint joint_4: axis 0 0 0 -> -1 0 0; limit lower=0 upper=0.03 effort=50 velocity=0.02 -> lower=0 upper=0.014 effort=50 velocity=0.02
- joint joint_5: axis 0 0 0 ->  1 0 0; limit lower=-0.03 upper=0 effort=50 velocity=0.02 -> lower=-0.014 upper=0 effort=50 velocity=0.02

Commit message: AGV nodes

File: src/nova_arm/urdf/nova_arm.urdf (robot description, URDF)
Before this commit: robot nova_arm, 6 links, 5 joints
Links:
- link Link_1: geometry collision mesh filename=package://nova_arm/meshes/Link_1.STL; visual mesh filename=package://nova_arm/meshes/Link_1.STL
- link Link_2: geometry collision mesh filename=package://nova_arm/meshes/Link_2.STL; visual mesh filename=package://nova_arm/meshes/Link_2.STL
- link Link_3: geometry collision mesh filename=package://nova_arm/meshes/Link_3.STL; visual mesh filename=package://nova_arm/meshes/Link_3.STL
- link Link_4: geometry collision mesh filename=package://nova_arm/meshes/Link_4.STL; visual mesh filename=package://nova_arm/meshes/Link_4.STL
- link Link_5: geometry collision mesh filename=package://nova_arm/meshes/Link_5.STL; visual mesh filename=package://nova_arm/meshes/Link_5.STL
- link base_link: geometry collision mesh filename=package://nova_arm/meshes/base_link.STL; visual mesh filename=package://nova_arm/meshes/base_link.STL
Joints:
- joint joint_2: limit lower=-1.5708 upper=1.5708 effort=12 velocity=1 -> lower=-1.919 upper=1.919 effort=12 velocity=1

Commit message: working inverse kinematics with micro-ros

File: src/nova_arm/urdf/nova_arm.urdf (robot description, URDF)
Before this commit: robot nova_arm, 6 links, 5 joints
Joints:
- removed joint joint_1
- removed joint joint_2
- removed joint joint_3
- added joint base_joint: type revolute, parent base_link, child Link_1, origin xyz=0 0  0.085 rpy=0 0 0, axis 0 0 1, limit lower=-3.1416 upper=3.1416 effort=15 velocity=1
- added joint elbow_joint: type revolute, parent Link_2, child Link_3, origin xyz=0.20 0 0 rpy=0 0 0, axis 0 0 1, limit lower=-2.332 upper=2.332 effort=10 velocity=1.5
- added joint shoulder_joint: type revolute, parent Link_1, child Link_2, origin xyz=0 0 0.066 rpy=0 -1.5708 0, axis 0 0 1, limit lower=-1.919 upper=1.919 effort=12 velocity=1
