Commit message: add hw ik node

File: src/nova/urdf/nova.urdf (robot description, URDF)
Before this commit: robot nova, 19 links, 18 joints
Joints:
- joint arm_mount_joint: origin xyz=0.175 0.0 0.125 rpy=-1.5708 3.14 0 -> xyz=0.175 0.0 0.125 rpy=-1.5708 3.1416 0
- joint joint_4: origin xyz=0.17556 0.0027305 -0.012575 rpy=1.5708 0 1.5708 -> xyz=0.17556 0.0023305 0.0 rpy=0 1.5708 0
- joint joint_5: origin xyz=0.17556 0.0018695 0.012575 rpy=-1.5708 0 -1.5708 -> xyz=0.17556 0.0022695 0.006 rpy=3.1416 -1.5708 0

Commit message: Resolve conflicts after rebase

File: src/nova/urdf/nova.urdf (robot description, URDF)
Before this commit: robot nova, 19 links, 18 joints
Joints:
- removed joint joint_1
- removed joint joint_2
- removed joint joint_3
- added joint arm_base_link: type revolute, parent base_link, child Link_1, origin xyz=0 0  0.085 rpy=0 0 0, axis 0 0 1, limit lower=-3.1416 upper=3.1416 effort=15 velocity=1
- added joint elbow_joint: type revolute, parent Link_2, child Link_3, origin xyz=0.20 0 0 rpy=0 0 0, axis 0 0 1, limit lower=-2.332 upper=2.332 effort=10 velocity=1.5
- added joint shoulder_joint: type revolute, parent Link_1, child Link_2, origin xyz=0 0 0.066 rpy=0 -1.5708 0, axis 0 0 1, limit lower=-1.919 upper=1.919 effort=12 velocity=1
- joint joint_4: origin xyz=0.17556 0.0023305 0.0 rpy=0 1.5708 0 -> xyz=0.17556 0.0027305 -0.012575 rpy=1.5708 0 1.5708
- joint joint_5: origin xyz=0.17556 0.0022695 0.006 rpy=3.1416 -1.5708 0 -> xyz=0.17556 0.0018695 0.012575 rpy=-1.5708 0 -1.5708

File: src/nova_arm/urdf/nova_arm.urdf (robot description, URDF)
Before this commit: robot nova_arm, 6 links, 5 joints
Links:
- removed link base_link
- added link arm_base_link, mass 0.7735; collision mesh filename=package://nova_arm/meshes/base_link.STL; visual mesh filename=package://nova_arm/meshes/base_link.STL
Joints:
- removed joint base_joint
- added joint arm_base_link: type revolute, parent base_link, child Link_1, origin xyz=0 0  0.085 rpy=0 0 0, axis 0 0 1, limit lower=-3.1416 upper=3.1416 effort=15 velocity=1
